Commit message: added colors

File: urdf/materials.xacro (robot description, xacro)
@@ -1,3 +1,24 @@
 <?xml version="1.0"?>
 <robot xmlns:xacro="http://www.ros.org/wiki/xacro">
+    <material name="grey">
+        <color rgba="0.5 0.5 0.5 1"/>
+    </material>
+    <material name="yellow">
+        <color rgba="1 1 0 1"/>
+    </material>
+    <material name="black">
+        <color rgba="0 0 0 1"/>
+    </material>
+    <material name="white">
+        <color rgba="1 1 1 1" />
+    </material>
+    <material name="orange">
+        <color rgba="1 0.3 0.1 1"/>
+    </material>
+    <material name="blue">
+        <color rgba="0.2 0.2 1 1"/>
+    </material>
+    <material name="red">
+        <color rgba="1 0 0 1"/>
+    </material>
 </robot>

File: urdf/robot_core.xacro (robot description, xacro)
@@ -15,4 +15,5 @@
                 <mesh   filename="file://$(find AMR-Sweeper_description)/meshes/Chassis/Chassis.stl" />
             </geometry>
+            <material name="grey"/>
         </visual>
         <collision>
@@ -40,4 +41,5 @@
                 <mesh   filename="file://$(find AMR-Sweeper_description)/meshes/WheelAssembly/WheelAssembly.stl" />
             </geometry>
+            <material name="yellow"/>
         </visual>
         <collision>
@@ -65,4 +67,5 @@
                 <mesh   filename="file://$(find AMR-Sweeper_description)/meshes/WheelAssembly/WheelAssembly.stl" />
             </geometry>
+            <material name="yellow"/>
         </visual>
         <collision>
@@ -89,4 +92,5 @@
             <!--    <mesh   filename="file://$(find AMR-Sweeper_description)/meshes/Sensors/GNSS.stl" />  -->
             </geometry>
+            <material name="black"/>
         </visual>
         <collision>
