Commit message: update

File: urdf/AMR-Sweeper.urdf.xacro (robot description, xacro)
@@ -3,4 +3,13 @@
     <xacro:include filename="robot_core.xacro" />
     <xacro:include filename="materials.xacro" />
+    <xacro:arg name="use_ros2_control" default="true"/>
+    <xacro:arg name="sim_mode" default="false"/>
     <xacro:include filename="gazebo_control.xacro" />
+    <xacro:include filename="ros2_control.xacro" />
+    <xacro:if value="$(arg use_ros2_control)">
+        <xacro:include filename="ros2_control.xacro" />
+    </xacro:if>
+    <xacro:unless value="$(arg use_ros2_control)">
+        <xacro:include filename="gazebo_control.xacro" />
+    </xacro:unless>
 </robot>

File: urdf/gazebo_control.xacro (robot description, xacro)
@@ -4,6 +4,6 @@
         <plugin name="gz::sim::systems::DiffDrive" filename="gz-sim-diff-drive.so">
             <!-- Wheel Information -->
-            <left_joint>left_wheel_joint</left_joint>
-            <right_joint>right_wheel_joint</right_joint>
+            <left_joint>LeftWheel_joint</left_joint>
+            <right_joint>RightWheel_joint</right_joint>
             <wheel_separation>0.244</wheel_separation>
             <wheel_radius>0.130</wheel_radius>
@@ -20,9 +20,9 @@
             <tf_topic>/tf</tf_topic>
         </plugin>
-        <plugin filename="gz-sim-join-state-publisher-system"
+        <plugin filename="gz-sim-joint-state-publisher-system"
               name="gz::sim::systems::JointStatePublisher">
                 <topic>joint_states</topic>
-                <joint_name>left_wheel_joint</joint_name>
-                <joint_name>right_wheel_joint</joint_name>
+                <joint_name>LeftWheel_joint</joint_name>
+                <joint_name>RightWheel_joint</joint_name>
         </plugin>
     </gazebo>

File: urdf/ros2_control.xacro (robot description, xacro)
@@ -5,6 +5,6 @@
             <hardware>
                 <plugin>diffdrive_arduino/DiffDriveArduino</plugin>
-                <param name="left_wheel_name">left_wheel_joint</param>
-                <param name="right_wheel_name">right_wheel_joint</param>
+                <param name="left_wheel_name">LeftWheel_joint</param>
+                <param name="right_wheel_name">RightWheel_joint</param>
                 <param name="loop_rate">30</param>
                 <param name="device">/dev/ttyUSB0</param>
@@ -36,5 +36,5 @@
                 <plugin>gz_ros2_control/GazeboSimSystem</plugin>
             </hardware>
-            <joint name="left_wheel_joint">
+            <joint name="LeftWheel_joint">
                 <command_interface name="velocity">
                     <param name="min">-10</param>
@@ -44,5 +44,5 @@
                 <state_interface name="position"/>
             </joint>
-            <joint name="right_wheel_joint">
+            <joint name="RightWheel_joint">
                 <command_interface name="velocity">
                     <param name="min">-10</param>
@@ -56,6 +56,6 @@
     <gazebo>
         <plugin name="gz_ros2_control::GazeboSimROS2ControlPlugin" filename="libgz_ros2_control-system.so">
-            <parameters>$(find articubot_one)/config/my_controllers.yaml</parameters>
-            <parameters>$(find articubot_one)/config/gaz_ros2_ctl_use_sim.yaml</parameters>
+            <parameters>$(find AMR-Sweeper_description)/config/controllers.yaml</parameters>
+            <parameters>$(find AMR-Sweeper_description)/config/gaz_ros2_ctl_use_sim.yaml</parameters>
         </plugin>
     </gazebo>

Commit message: update

File: urdf/AMR-Sweeper.urdf.xacro (robot description, xacro)
@@ -2,9 +2,5 @@
 <robot xmlns:xacro="http://www.ros.org/wiki/xacro"  name="AMRSweeper">
     <xacro:include filename="robot_core.xacro" />
-    <xacro:include filename="materials.xacro" />
     <xacro:arg name="use_ros2_control" default="true"/>
-    <xacro:arg name="sim_mode" default="false"/>
-    <xacro:include filename="gazebo_control.xacro" />
-    <xacro:include filename="ros2_control.xacro" />
     <xacro:if value="$(arg use_ros2_control)">
         <xacro:include filename="ros2_control.xacro" />
@@ -13,3 +9,4 @@
         <xacro:include filename="gazebo_control.xacro" />
     </xacro:unless>
+    <xacro:arg name="sim_mode" default="false"/>
 </robot>

File: urdf/robot_core.xacro (robot description, xacro)
@@ -1,4 +1,5 @@
 <?xml version="1.0"?>
 <robot xmlns:xacro="http://www.ros.org/wiki/xacro">
+    <xacro:include filename="materials.xacro" />
     <link name="base_link">
     </link>

File: urdf/ros2_control.xacro (robot description, xacro)
@@ -1,62 +1,31 @@
 <?xml version="1.0"?>
 <robot xmlns:xacro="http://www.ros.org/wiki/xacro">
-    <xacro:unless value="$(arg sim_mode)">
-        <ros2_control name="RealRobot" type="system">
-            <hardware>
-                <plugin>diffdrive_arduino/DiffDriveArduino</plugin>
-                <param name="left_wheel_name">LeftWheel_joint</param>
-                <param name="right_wheel_name">RightWheel_joint</param>
-                <param name="loop_rate">30</param>
-                <param name="device">/dev/ttyUSB0</param>
-                <param name="baud_rate">57600</param>
-                <param name="timeout">1000</param>
-                <param name="enc_counts_per_rev">3436</param>
-            </hardware>
-            <joint name="LeftWheel_joint">
-                <command_interface name="velocity">
-                    <param name="min">-10</param>
-                    <param name="max">10</param>
-                </command_interface>
-                <state_interface name="velocity"/>
-                <state_interface name="position"/>
-            </joint>
-            <joint name="RightWheel_joint">
-                <command_interface name="velocity">
-                    <param name="min">-10</param>
-                    <param name="max">10</param>
-                </command_interface>
-                <state_interface name="velocity"/>
-                <state_interface name="position"/>
-            </joint>
-        </ros2_control>
-    </xacro:unless>
-    <xacro:if value="$(arg sim_mode)">
-        <ros2_control name="GazeboSystem" type="system">
-            <hardware>
-                <plugin>gz_ros2_control/GazeboSimSystem</plugin>
-            </hardware>
-            <joint name="LeftWheel_joint">
-                <command_interface name="velocity">
-                    <param name="min">-10</param>
-                    <param name="max">10</param>
-                </command_interface>
-                <state_interface name="velocity"/>
-                <state_interface name="position"/>
-            </joint>
-            <joint name="RightWheel_joint">
-                <command_interface name="velocity">
-                    <param name="min">-10</param>
-                    <param name="max">10</param>
-                </command_interface>
-                <state_interface name="velocity"/>
-                <state_interface name="position"/>
-            </joint>
-        </ros2_control>
-    </xacro:if>
-    <gazebo>
-        <plugin name="gz_ros2_control::GazeboSimROS2ControlPlugin" filename="libgz_ros2_control-system.so">
-            <parameters>$(find AMR-Sweeper_description)/config/controllers.yaml</parameters>
-            <parameters>$(find AMR-Sweeper_description)/config/gaz_ros2_ctl_use_sim.yaml</parameters>
-        </plugin>
-    </gazebo>
+    <ros2_control name="RealRobot" type="system">
+        <hardware>
+            <plugin>diffdrive_arduino/DiffDriveArduino</plugin>
+            <param name="left_wheel_name">LeftWheel_joint</param>
+            <param name="right_wheel_name">RightWheel_joint</param>
+            <param name="loop_rate">30</param>
+            <param name="device">/dev/ttyUSB0</param>
+            <param name="baud_rate">57600</param>
+            <param name="timeout">1000</param>
+            <param name="enc_counts_per_rev">3436</param>
+        </hardware>
+        <joint name="LeftWheel_joint">
+            <command_interface name="velocity">
+                <param name="min">-10</param>
+                <param name="max">10</param>
+            </command_interface>
+            <state_interface name="velocity"/>
+            <state_interface name="position"/>
+        </joint>
+        <joint name="RightWheel_joint">
+            <command_interface name="velocity">
+                <param name="min">-10</param>
+                <param name="max">10</param>
+            </command_interface>
+            <state_interface name="velocity"/>
+            <state_interface name="position"/>
+        </joint>
+    </ros2_control>
 </robot>

Commit message: added RVIZ2 launch and GNSS sensor

File: urdf/AMR-Sweeper.urdf.xacro (robot description, xacro)
@@ -2,4 +2,5 @@
 <robot xmlns:xacro="http://www.ros.org/wiki/xacro"  name="AMRSweeper">
     <xacro:include filename="robot_core.xacro" />
+    <xacro:include filename="sensors.xacro" />
     <xacro:arg name="use_ros2_control" default="true"/>
     <xacro:if value="$(arg use_ros2_control)">

File: urdf/robot_core.xacro (robot description, xacro)
@@ -78,3 +78,27 @@
         </inertial>
     </link>
+    <joint name="GNSS_joint" type="fixed">
+        <parent link="base_link" />
+        <child  link="GNSS_link" />
+        <origin xyz="0 0 0" rpy="0 0 0"/>
+    </joint>
+    <link name="GNSS_link">
+        <visual>
+            <origin xyz="0 0 0" rpy="0 0 0"/>
+            <geometry>
+            <!--    <mesh   filename="file://$(find AMR-Sweeper_description)/meshes/Sensors/GNSS.stl" />  -->
+            </geometry>
+        </visual>
+        <collision>
+            <origin xyz="0 0 0" rpy="0 0 0"/>
+            <geometry>
+            <!--    <mesh   filename="file://$(find AMR-Sweeper_description)/meshes/Sensors/GNSS.stl" />  -->
+            </geometry>
+        </collision>
+        <inertial>
+            <origin xyz="0 0 0" rpy="0 0 0"/>
+            <mass value="0" />
+            <inertia ixx="0" ixy="0" ixz="0" iyy="0" iyz="0" izz="0" />
+        </inertial>
+    </link>
 </robot>

Commit message: added camera

File: urdf/AMR-Sweeper.urdf.xacro (robot description, xacro)
@@ -1,6 +1,8 @@
 <?xml version="1.0"?>
 <robot xmlns:xacro="http://www.ros.org/wiki/xacro"  name="AMRSweeper">
+    <xacro:include filename="materials.xacro" />
     <xacro:include filename="robot_core.xacro" />
-    <xacro:include filename="sensors.xacro" />
+    <xacro:include filename="GNSS_sensor.xacro" />
+    <xacro:include filename="depth_camera.xacro" />
     <xacro:arg name="use_ros2_control" default="true"/>
     <xacro:if value="$(arg use_ros2_control)">

File: urdf/robot_core.xacro (robot description, xacro)
@@ -1,5 +1,4 @@
 <?xml version="1.0"?>
 <robot xmlns:xacro="http://www.ros.org/wiki/xacro">
-    <xacro:include filename="materials.xacro" />
     <link name="base_link">
     </link>
@@ -81,28 +80,3 @@
         </inertial>
     </link>
-    <joint name="GNSS_joint" type="fixed">
-        <parent link="base_link" />
-        <child  link="GNSS_link" />
-        <origin xyz="0 0 0" rpy="0 0 0"/>
-    </joint>
-    <link name="GNSS_link">
-        <visual>
-            <origin xyz="0 0 0" rpy="0 0 0"/>
-            <geometry>
-            <!--    <mesh   filename="file://$(find AMR-Sweeper_description)/meshes/Sensors/GNSS.stl" />  -->
-            </geometry>
-            <material name="black"/>
-        </visual>
-        <collision>
-            <origin xyz="0 0 0" rpy="0 0 0"/>
-            <geometry>
-            <!--    <mesh   filename="file://$(find AMR-Sweeper_description)/meshes/Sensors/GNSS.stl" />  -->
-            </geometry>
-        </collision>
-        <inertial>
-            <origin xyz="0 0 0" rpy="0 0 0"/>
-            <mass value="0" />
-            <inertia ixx="0" ixy="0" ixz="0" iyy="0" iyz="0" izz="0" />
-        </inertial>
-    </link>
 </robot>
