Commit message: Update depth_camera.xacro

File: urdf/depth_camera.xacro (robot description, xacro)
@@ -13,4 +13,10 @@
             <material name="red"/>
         </visual>
+        <collision>
+            <origin xyz="0 0 0" rpy="0 0 0"/>
+            <geometry>
+                <box size="0.010 0.03 0.5"/>
+            </geometry>
+        </collision>
     </link>
     <joint name="camera_optical_joint" type="fixed">

Commit message: Update depth_camera.xacro

File: urdf/depth_camera.xacro (robot description, xacro)
@@ -13,17 +13,5 @@
             <material name="red"/>
         </visual>
-        <collision>
-            <origin xyz="0 0 0" rpy="0 0 0"/>
-            <geometry>
-                <box size="0.010 0.03 0.5"/>
-            </geometry>
-        </collision>
     </link>
-    <joint name="camera_optical_joint" type="fixed">
-        <parent link="camera_link"/>
-        <child link="camera_link_optical"/>
-        <origin xyz="0 0 0" rpy="${-pi/2} 0 ${-pi/2}"/>
-    </joint>
-    <link name="camera_link_optical"></link>
     <gazebo reference="camera_link">
         <sensor name="depth_camera" type="depth_camera">
@@ -65,3 +53,9 @@
         </sensor>
     </gazebo>
+    <joint name="camera_optical_joint" type="fixed">
+        <parent link="camera_link"/>
+        <child link="camera_link_optical"/>
+        <origin xyz="0 0 0" rpy="${-pi/2} 0 ${-pi/2}"/>
+    </joint>
+    <link name="camera_link_optical"></link>
 </robot>

Commit message: Update depth_camera.xacro

File: urdf/depth_camera.xacro (robot description, xacro)
@@ -13,5 +13,4 @@
             <material name="red"/>
         </visual>
-    </link>
     <gazebo reference="camera_link">
         <sensor name="depth_camera" type="depth_camera">
@@ -53,4 +52,5 @@
         </sensor>
     </gazebo>
+    </link>
     <joint name="camera_optical_joint" type="fixed">
         <parent link="camera_link"/>

Commit message: Update depth_camera.xacro

File: urdf/depth_camera.xacro (robot description, xacro)
@@ -13,4 +13,12 @@
             <material name="red"/>
         </visual>
+    </link>
+    <joint name="camera_optical_joint" type="fixed">
+        <parent link="camera_link"/>
+        <child link="camera_link_optical"/>
+        <origin xyz="0 0 0" rpy="${-pi/2} 0 ${-pi/2}"/>
+    </joint>
+    <link name="camera_link_optical"></link>
+   <gazebo reference="camera_link">
         <sensor name="depth_camera" type="depth_camera">
             <update_rate>10</update_rate>
@@ -29,4 +37,6 @@
             </camera>
         </sensor>
+    </gazebo>
+    <gazebo reference="camera_link">
         <sensor name="camera" type="camera">
             <pose> 0 0 0 0 0 0 </pose>
@@ -48,10 +58,4 @@
             <topic>camera/image_raw</topic>
         </sensor>
-    </link>
-    <joint name="camera_optical_joint" type="fixed">
-        <parent link="camera_link"/>
-        <child link="camera_link_optical"/>
-        <origin xyz="0 0 0" rpy="${-pi/2} 0 ${-pi/2}"/>
-    </joint>
-    <link name="camera_link_optical"></link>
+    </gazebo>
 </robot>

Commit message: updated base_link to base_footprint

File: urdf/depth_camera.xacro (robot description, xacro)
@@ -13,43 +13,4 @@
             <material name="red"/>
         </visual>
-        <gazebo reference="camera_link">
-            <sensor name="depth_camera" type="depth_camera">
-                <update_rate>10</update_rate>
-                <topic>depth_camera</topic>
-                <camera>
-                    <horizontal_fov>1.05</horizontal_fov>
-                    <image>
-                        <width>256</width>
-                        <height>256</height>
-                        <format>R_FLOAT32</format>
-                    </image>
-                    <clip>
-                        <near>0.1</near>
-                        <far>10.0</far>
-                    </clip>
-                </camera>
-            </sensor>
-        </gazebo>
-        <gazebo reference="camera_link">
-            <sensor name="camera" type="camera">
-                <pose> 0 0 0 0 0 0 </pose>
-                <visualize>true</visualize>
-                <update_rate>10</update_rate>
-                <camera>
-                    <camera_info_topic>camera/camera_info</camera_info_topic>
-                    <horizontal_fov>1.089</horizontal_fov>
-                    <image>
-                        <format>R8G8B8</format>
-                        <width>640</width>
-                        <height>480</height>
-                    </image>
-                    <clip>
-                        <near>0.05</near>
-                        <far>8.0</far>
-                    </clip>
-                </camera>
-                <topic>camera/image_raw</topic>
-            </sensor>
-        </gazebo>
     </link>
     <joint name="camera_optical_joint" type="fixed">
@@ -59,3 +20,42 @@
     </joint>
     <link name="camera_link_optical"></link>
+   <gazebo reference="camera_link">
+        <sensor name="depth_camera" type="depth_camera">
+            <update_rate>10</update_rate>
+            <topic>depth_camera</topic>
+            <camera>
+                <horizontal_fov>1.05</horizontal_fov>
+                <image>
+                    <width>256</width>
+                    <height>256</height>
+                    <format>R_FLOAT32</format>
+                </image>
+                <clip>
+                    <near>0.1</near>
+                    <far>10.0</far>
+                </clip>
+            </camera>
+        </sensor>
+    </gazebo>
+    <gazebo reference="camera_link">
+        <sensor name="camera" type="camera">
+            <pose> 0 0 0 0 0 0 </pose>
+            <visualize>true</visualize>
+            <update_rate>10</update_rate>
+            <camera>
+                <camera_info_topic>camera/camera_info</camera_info_topic>
+                <horizontal_fov>1.089</horizontal_fov>
+                <image>
+                    <format>R8G8B8</format>
+                    <width>640</width>
+                    <height>480</height>
+                </image>
+                <clip>
+                    <near>0.05</near>
+                    <far>8.0</far>
+                </clip>
+            </camera>
+            <topic>camera/image_raw</topic>
+        </sensor>
+    </gazebo>
 </robot>

File: urdf/gazebo_control.xacro (robot description, xacro)
@@ -17,5 +17,5 @@
             <!-- Output -->
             <frame_id>odom</frame_id>
-            <child_frame_id>base_link</child_frame_id>
+            <child_frame_id>base_footprint</child_frame_id>
             <odom_topic>odom</odom_topic>
             <odom_publisher_frequency>30</odom_publisher_frequency>

File: urdf/robot_core.xacro (robot description, xacro)
@@ -1,12 +1,12 @@
 <?xml version="1.0"?>
 <robot xmlns:xacro="http://www.ros.org/wiki/xacro">
-    <link name="base_link">
+    <link name="base_footprint">
     </link>
-    <joint name="base_footprint_joint" type="fixed">
-        <parent link="base_link" />
-        <child  link="base_footprint" />
+    <joint name="base_link_joint" type="fixed">
+        <parent link="base_footprint" />
+        <child  link="base_link" />
         <origin xyz="0 0 -0.13" rpy="0 0 0"/>
     </joint>
-    <link name="base_footprint">
+    <link name="base_link">
     </link>
     <joint name="Chassis_joint" type="fixed">
