Commit message: update to aunch gz_sim

File: urdf/gazebo_control.xacro (robot description, xacro)
@@ -2,5 +2,5 @@
 <robot xmlns:xacro="http://www.ros.org/wiki/xacro">
     <gazebo>
-        <plugin name="gz::sim::systems::DiffDrive" filename="gz-sim-diff-drive.so">
+        <plugin name="gz::sim::systems::DiffDrive" filename="gz-sim-diff-drive-system">
             <!-- Wheel Information -->
             <left_joint>LeftWheel_joint</left_joint>

File: urdf/robot_core.xacro (robot description, xacro)
@@ -2,4 +2,11 @@
 <robot xmlns:xacro="http://www.ros.org/wiki/xacro">
     <link name="base_link">
+    </link>
+    <joint name="Chassis_joint" type="fixed">
+        <parent link="base_link" />
+        <child  link="Chassis_link" />
+        <origin xyz="0 0 0" rpy="0 0 0"/>
+    </joint>
+    <link name="Chassis_link">
         <visual>
             <origin xyz="0 0 0" rpy="0 0 0"/>

Commit message: update

File: urdf/gazebo_control.xacro (robot description, xacro)
@@ -8,5 +8,5 @@
             <left_joint>LeftWheel_joint</left_joint>
             <right_joint>RightWheel_joint</right_joint>
-            <wheel_separation>0.244</wheel_separation>
+            <wheel_separation>0.488</wheel_separation>
             <wheel_radius>0.130</wheel_radius>
             <!-- Limits -->

File: urdf/robot_core.xacro (robot description, xacro)
@@ -23,4 +23,5 @@
             <material name="grey"/>
         </visual>
+<!--
         <collision>
             <origin xyz="0 0 0" rpy="0 0 0"/>
@@ -29,4 +30,5 @@
             </geometry>
         </collision>
+-->
         <inertial>
             <origin xyz="0.054 0 0.110" rpy="0 0 0"/>
@@ -52,5 +54,5 @@
             <origin xyz="0 0 0" rpy="${pi/2} 0 0"/>
             <geometry>
-                <mesh   filename="file://$(find AMR-Sweeper_description)/meshes/WheelAssembly/WheelAssembly.stl" />
+                <cylinder radius="0.130" length="0.08"/>
             </geometry>
         </collision>
@@ -78,5 +80,5 @@
             <origin xyz="0 0 0" rpy="${pi/2} 0 0"/>
             <geometry>
-                <mesh   filename="file://$(find AMR-Sweeper_description)/meshes/WheelAssembly/WheelAssembly.stl" />
+                <cylinder radius="0.130" length="0.08"/>
             </geometry>
         </collision>
@@ -102,10 +104,4 @@
             <material name="black"/>
         </visual>
-        <collision>
-            <origin xyz="0 0 0" rpy="0 0 0"/>
-            <geometry>
-                <mesh   filename="file://$(find AMR-Sweeper_description)/meshes/Tool/Tool.stl" />
-            </geometry>
-        </collision>
         <inertial>
             <origin xyz="0 0 0" rpy="0 0 0"/>
