Commit message: Update robot_core.xacro
Removed scale factor

File: urdf/robot_core.xacro (robot description, xacro)
@@ -5,6 +5,5 @@
             <origin xyz="0 0 0" rpy="0 0 0"/>
             <geometry>
-                <mesh   filename="file://$(find AMR-Sweeper)/meshes/BottomAssembly/MotorAssembly.stl"
-                        scale="0.001 0.001 0.001" />
+                <mesh   filename="file://$(find AMR-Sweeper)/meshes/BottomAssembly/MotorAssembly.stl" />
             </geometry>
         </visual>
@@ -20,6 +19,5 @@
             <origin xyz="0 0 0" rpy="0 0 0"/>
             <geometry>
-                <mesh   filename="file://$(find AMR-Sweeper)/meshes/BottomAssembly/WheelAssembly.stl"
-                        scale="0.001 0.001 0.001" />
+                <mesh   filename="file://$(find AMR-Sweeper)/meshes/BottomAssembly/WheelAssembly.stl" />
             </geometry>
         </visual>
@@ -35,6 +33,5 @@
             <origin xyz="0 0 0" rpy="0 0 0"/>
             <geometry>
-                <mesh   filename="file://$(find AMR-Sweeper)/meshes/BottomAssembly/WheelAssembly.stl"
-                        scale="0.001 0.001 0.001" />
+                <mesh   filename="file://$(find AMR-Sweeper)/meshes/BottomAssembly/WheelAssembly.stl" />
             </geometry>
         </visual>

Commit message: Update robot_core.xacro
updated offset

File: urdf/robot_core.xacro (robot description, xacro)
@@ -13,5 +13,5 @@
         <child  link="LeftWheel_link" />
         <axis   xyz="0 0 1" />
-        <origin xyz="0 0.2626 0" rpy="-${pi/2} 0 0" />
+        <origin xyz="0 0.244 0" rpy="-${pi/2} 0 0" />
     </joint>
     <link name="LeftWheel_link">
@@ -27,5 +27,5 @@
         <child  link="RightWheel_link" />
         <axis   xyz="0 0 1" />
-        <origin xyz="0 -0.2626 0" rpy="${pi/2} 0 0" />
+        <origin xyz="0 -0.244 0" rpy="${pi/2} 0 0" />
     </joint>
     <link name="RightWheelAssembly_link">

Commit message: Update robot_core.xacro

File: urdf/robot_core.xacro (robot description, xacro)
@@ -29,5 +29,5 @@
         <origin xyz="0 -0.244 0" rpy="${pi/2} 0 0" />
     </joint>
-    <link name="RightWheelAssembly_link">
+    <link name="RightWheel_link">
         <visual>
             <origin xyz="0 0 0" rpy="0 0 0"/>
@@ -37,3 +37,31 @@
         </visual>
     </link>
+    <joint name="MiddleAssembly_joint" type="fixed">
+        <parent link="base_link" />
+        <child  link="MiddleAssembly_link" />
+        <axis   xyz="0 0 1" />
+        <origin xyz="0 -0.244 0" rpy="${pi/2} 0 0" />
+    </joint>
+    <link name="MiddleAssembly_link">
+        <visual>
+            <origin xyz="0 0 0" rpy="0 0 0"/>
+            <geometry>
+                <mesh   filename="file://$(find AMR-Sweeper)/meshes/MiddleAssembly/ChassisAssembly.stl" />
+            </geometry>
+        </visual>
+    </link>
+    <joint name="TopAssembly_joint" type="fixed">
+        <parent link="base_link" />
+        <child  link="TopAssembly_link" />
+        <axis   xyz="0 0 1" />
+        <origin xyz="0 -0.244 0" rpy="${pi/2} 0 0" />
+    </joint>
+    <link name="TopAssembly_link">
+        <visual>
+            <origin xyz="0 0 0" rpy="0 0 0"/>
+            <geometry>
+                <mesh   filename="file://$(find AMR-Sweeper)/meshes/TopAssembly/TopAssembly.stl" />
+            </geometry>
+        </visual>
+    </link>
 </robot>

Commit message: Update robot_core.xacro

File: urdf/robot_core.xacro (robot description, xacro)
@@ -5,5 +5,5 @@
             <origin xyz="0 0 0" rpy="0 0 0"/>
             <geometry>
-                <mesh   filename="file://$(find AMR-Sweeper)/meshes/BottomAssembly/MotorAssembly.stl" />
+                <mesh   filename="file://$(find AMR-Sweeper_description)/meshes/Chassis/Chassis.stl" />
             </geometry>
         </visual>
@@ -19,5 +19,5 @@
             <origin xyz="0 0 0" rpy="0 0 0"/>
             <geometry>
-                <mesh   filename="file://$(find AMR-Sweeper)/meshes/BottomAssembly/WheelAssembly.stl" />
+                <mesh   filename="file://$(find AMR-Sweeper_description)/meshes/WheelAssembly/WheelAssembly.stl" />
             </geometry>
         </visual>
@@ -26,5 +26,5 @@
         <parent link="base_link" />
         <child  link="RightWheel_link" />
-        <axis   xyz="0 0 1" />
+        <axis   xyz="0 0 -1" />
         <origin xyz="0 -0.244 0" rpy="${pi/2} 0 0" />
     </joint>
@@ -33,33 +33,5 @@
             <origin xyz="0 0 0" rpy="0 0 0"/>
             <geometry>
-                <mesh   filename="file://$(find AMR-Sweeper)/meshes/BottomAssembly/WheelAssembly.stl" />
-            </geometry>
-        </visual>
-    </link>
-    <joint name="MiddleAssembly_joint" type="fixed">
-        <parent link="base_link" />
-        <child  link="MiddleAssembly_link" />
-        <axis   xyz="0 0 1" />
-        <origin xyz="0 -0.244 0" rpy="${pi/2} 0 0" />
-    </joint>
-    <link name="MiddleAssembly_link">
-        <visual>
-            <origin xyz="0 0 0" rpy="0 0 0"/>
-            <geometry>
-                <mesh   filename="file://$(find AMR-Sweeper)/meshes/MiddleAssembly/ChassisAssembly.stl" />
-            </geometry>
-        </visual>
-    </link>
-    <joint name="TopAssembly_joint" type="fixed">
-        <parent link="base_link" />
-        <child  link="TopAssembly_link" />
-        <axis   xyz="0 0 1" />
-        <origin xyz="0 -0.244 0" rpy="${pi/2} 0 0" />
-    </joint>
-    <link name="TopAssembly_link">
-        <visual>
-            <origin xyz="0 0 0" rpy="0 0 0"/>
-            <geometry>
-                <mesh   filename="file://$(find AMR-Sweeper)/meshes/TopAssembly/TopAssembly.stl" />
+                <mesh   filename="file://$(find AMR-Sweeper_description)/meshes/WheelAssembly/WheelAssembly.stl" />
             </geometry>
         </visual>

Commit message: update

File: urdf/robot_core.xacro (robot description, xacro)
@@ -3,5 +3,5 @@
     <link name="base_link">
         <visual>
-            <origin xyz="0 0 0" rpy="0 0 0"/>
+            <origin xyz="0 0 0.130" rpy="0 0 0"/>
             <geometry>
                 <mesh   filename="file://$(find AMR-Sweeper_description)/meshes/Chassis/Chassis.stl" />

Commit message: update

File: urdf/robot_core.xacro (robot description, xacro)
@@ -3,5 +3,5 @@
     <link name="base_link">
         <visual>
-            <origin xyz="0 0 0.130" rpy="0 0 0"/>
+            <origin xyz="0 0 0" rpy="0 0 0"/>
             <geometry>
                 <mesh   filename="file://$(find AMR-Sweeper_description)/meshes/Chassis/Chassis.stl" />
@@ -12,6 +12,6 @@
         <parent link="base_link" />
         <child  link="LeftWheel_link" />
+        <origin xyz="0 0.244 0" rpy="-${pi/2} 0 0" />
         <axis   xyz="0 0 1" />
-        <origin xyz="0 0.244 0" rpy="-${pi/2} 0 0" />
     </joint>
     <link name="LeftWheel_link">
@@ -26,6 +26,6 @@
         <parent link="base_link" />
         <child  link="RightWheel_link" />
+        <origin xyz="0 -0.244 0" rpy="${pi/2} 0 0" />
         <axis   xyz="0 0 -1" />
-        <origin xyz="0 -0.244 0" rpy="${pi/2} 0 0" />
     </joint>
     <link name="RightWheel_link">

Commit message: update

File: urdf/robot_core.xacro (robot description, xacro)
@@ -17,5 +17,5 @@
     <link name="LeftWheel_link">
         <visual>
-            <origin xyz="0 0 0" rpy="0 0 0"/>
+            <origin xyz="0 0 0" rpy="-${pi/2} 0 0"/>
             <geometry>
                 <mesh   filename="file://$(find AMR-Sweeper_description)/meshes/WheelAssembly/WheelAssembly.stl" />
@@ -31,5 +31,5 @@
     <link name="RightWheel_link">
         <visual>
-            <origin xyz="0 0 0" rpy="0 0 0"/>
+            <origin xyz="0 0 0" rpy="${pi/2} 0 0"/>
             <geometry>
                 <mesh   filename="file://$(find AMR-Sweeper_description)/meshes/WheelAssembly/WheelAssembly.stl" />

Commit message: update

File: urdf/robot_core.xacro (robot description, xacro)
@@ -17,5 +17,5 @@
     <link name="LeftWheel_link">
         <visual>
-            <origin xyz="0 0 0" rpy="-${pi/2} 0 0"/>
+            <origin xyz="0 0 0" rpy="${pi/2} 0 0"/>
             <geometry>
                 <mesh   filename="file://$(find AMR-Sweeper_description)/meshes/WheelAssembly/WheelAssembly.stl" />

Commit message: gz_sim launch updated

File: urdf/robot_core.xacro (robot description, xacro)
@@ -8,4 +8,15 @@
             </geometry>
         </visual>
+        <collision>
+            <origin xyz="0 0 0" rpy="0 0 0"/>
+            <geometry>
+                <mesh   filename="file://$(find AMR-Sweeper_description)/meshes/Chassis/Chassis.stl" />
+            </geometry>
+        </collision>
+        <inertial>
+            <origin xyz="0 0 0" rpy="0 0 0"/>
+            <mass value="5" />
+            <inertia ixx="1" ixy="0.0" ixz="0.0" iyy="1" iyz="0.0" izz="1" />
+        </inertial>
     </link>
     <joint name="LeftWheel_joint" type="continuous">
@@ -22,4 +33,15 @@
             </geometry>
         </visual>
+        <collision>
+            <origin xyz="0 0 0" rpy="${pi/2} 0 0"/>
+            <geometry>
+                <mesh   filename="file://$(find AMR-Sweeper_description)/meshes/WheelAssembly/WheelAssembly.stl" />
+            </geometry>
+        </collision>
+        <inertial>
+            <origin xyz="0 0 0" rpy="0 0 0"/>
+            <mass value="0.5" />
+            <inertia ixx="1" ixy="0.0" ixz="0.0" iyy="1" iyz="0.0" izz="1" />
+        </inertial>
     </link>
     <joint name="RightWheel_joint" type="continuous">
@@ -36,4 +58,15 @@
             </geometry>
         </visual>
+        <collision>
+            <origin xyz="0 0 0" rpy="${pi/2} 0 0"/>
+            <geometry>
+                <mesh   filename="file://$(find AMR-Sweeper_description)/meshes/WheelAssembly/WheelAssembly.stl" />
+            </geometry>
+        </collision>
+        <inertial>
+            <origin xyz="0 0 0" rpy="0 0 0"/>
+            <mass value="0.5" />
+            <inertia ixx="1" ixy="0.0" ixz="0.0" iyy="1" iyz="0.0" izz="1" />
+        </inertial>
     </link>
 </robot>

Commit message: Updated Inertia

File: urdf/robot_core.xacro (robot description, xacro)
@@ -15,7 +15,7 @@
         </collision>
         <inertial>
-            <origin xyz="0 0 0" rpy="0 0 0"/>
-            <mass value="5" />
-            <inertia ixx="1" ixy="0.0" ixz="0.0" iyy="1" iyz="0.0" izz="1" />
+            <origin xyz="0.054 0 0.110" rpy="0 0 0"/>
+            <mass value="15.4" />
+            <inertia ixx="0.2" ixy="0.002" ixz="-0.010" iyy="0.376" iyz="0.000" izz="0.508" />
         </inertial>
     </link>
@@ -40,7 +40,7 @@
         </collision>
         <inertial>
-            <origin xyz="0 0 0" rpy="0 0 0"/>
-            <mass value="0.5" />
-            <inertia ixx="1" ixy="0.0" ixz="0.0" iyy="1" iyz="0.0" izz="1" />
+            <origin xyz="0 0.1 0" rpy="0 0 0"/>
+            <mass value="1.5" />
+            <inertia ixx="0.01" ixy="0" ixz="0" iyy="0.02" iyz="0" izz="0.01" />
         </inertial>
     </link>
@@ -65,7 +65,7 @@
         </collision>
         <inertial>
-            <origin xyz="0 0 0" rpy="0 0 0"/>
-            <mass value="0.5" />
-            <inertia ixx="1" ixy="0.0" ixz="0.0" iyy="1" iyz="0.0" izz="1" />
+            <origin xyz="0 0.1 0" rpy="0 0 0"/>
+            <mass value="1.5" />
+            <inertia ixx="0.01" ixy="0" ixz="0" iyy="0.02" iyz="0" izz="0.01" />
         </inertial>
     </link>

Commit message: Update

File: urdf/robot_core.xacro (robot description, xacro)
@@ -2,4 +2,11 @@
 <robot xmlns:xacro="http://www.ros.org/wiki/xacro">
     <link name="base_link">
+    </link>
+    <joint name="base_footprint_joint" type="fixed">
+        <parent link="base_link" />
+        <child  link="base_footprint" />
+        <origin xyz="0 0 -0.13" rpy="0 0 0"/>
+    </joint>
+    <link name="base_footprint">
     </link>
     <joint name="Chassis_joint" type="fixed">

Commit message: Update robot_core.xacro

File: urdf/robot_core.xacro (robot description, xacro)
@@ -6,5 +6,5 @@
         <parent link="base_footprint" />
         <child  link="base_link" />
-        <origin xyz="0 0 -0.13" rpy="0 0 0"/>
+        <origin xyz="0 0 0.13" rpy="0 0 0"/>
     </joint>
     <link name="base_link">

Commit message: Added Tool

File: urdf/robot_core.xacro (robot description, xacro)
@@ -56,5 +56,5 @@
         </collision>
         <inertial>
-            <origin xyz="0 0.1 0" rpy="0 0 0"/>
+            <origin xyz="0 0 0" rpy="0 0 0"/>
             <mass value="1.5" />
             <inertia ixx="0.01" ixy="0" ixz="0" iyy="0.02" iyz="0" izz="0.01" />
@@ -82,8 +82,35 @@
         </collision>
         <inertial>
-            <origin xyz="0 0.1 0" rpy="0 0 0"/>
+            <origin xyz="0 0 0" rpy="0 0 0"/>
             <mass value="1.5" />
             <inertia ixx="0.01" ixy="0" ixz="0" iyy="0.02" iyz="0" izz="0.01" />
         </inertial>
     </link>
+    <joint name="Tool_joint" type="revolute">
+        <parent link="base_link" />
+        <child  link="Tool_link" />
+        <origin xyz="0 0 0.155" rpy="0 0 0" />
+        <axis   xyz="1 0 0" />
+        <limit  lower="-${pi/18}" upper="${pi/18}"/>
+    </joint>
+    <link name="Tool_link">
+        <visual>
+            <origin xyz="0 0 0" rpy="0 0 0"/>
+            <geometry>
+                <mesh   filename="file://$(find AMR-Sweeper_description)/meshes/Tool/Tool.stl" />
+            </geometry>
+            <material name="black"/>
+        </visual>
+        <collision>
+            <origin xyz="0 0 0" rpy="0 0 0"/>
+            <geometry>
+                <mesh   filename="file://$(find AMR-Sweeper_description)/meshes/Tool/Tool.stl" />
+            </geometry>
+        </collision>
+        <inertial>
+            <origin xyz="0 0 0" rpy="0 0 0"/>
+            <mass value="2.5" />
+            <inertia ixx="0.01" ixy="0" ixz="0" iyy="0.02" iyz="0" izz="0.01" />
+        </inertial>
+    </link>
 </robot>

Commit message: update

File: urdf/robot_core.xacro (robot description, xacro)
@@ -92,5 +92,5 @@
         <origin xyz="0 0 0.155" rpy="0 0 0" />
         <axis   xyz="1 0 0" />
-        <limit  lower="-${pi/18}" upper="${pi/18}"/>
+    <!--    <limit  lower="-${pi/18}" upper="${pi/18}"/>  -->
     </joint>
     <link name="Tool_link">

Commit message: update

File: urdf/robot_core.xacro (robot description, xacro)
@@ -92,5 +92,5 @@
         <origin xyz="0 0 0.155" rpy="0 0 0" />
         <axis   xyz="1 0 0" />
-    <!--    <limit  lower="-${pi/18}" upper="${pi/18}"/>  -->
+        <limit  lower="0" upper="${pi/2}"/>
     </joint>
     <link name="Tool_link">

Commit message: update

File: urdf/robot_core.xacro (robot description, xacro)
@@ -92,5 +92,5 @@
         <origin xyz="0 0 0.155" rpy="0 0 0" />
         <axis   xyz="1 0 0" />
-        <limit  lower="0" upper="${pi/2}"/>
+        <limit  lower="0" upper="${pi/2}" effort="100"/>
     </joint>
     <link name="Tool_link">

Commit message: update

File: urdf/robot_core.xacro (robot description, xacro)
@@ -92,5 +92,5 @@
         <origin xyz="0 0 0.155" rpy="0 0 0" />
         <axis   xyz="1 0 0" />
-        <limit  lower="0" upper="${pi/2}" effort="100"/>
+        <limit  lower="0" upper="${pi/2}" velocity="100" effort="100"/>
     </joint>
     <link name="Tool_link">

Commit message: update

File: urdf/robot_core.xacro (robot description, xacro)
@@ -90,7 +90,7 @@
         <parent link="base_link" />
         <child  link="Tool_link" />
-        <origin xyz="0 0 0.155" rpy="0 0 0" />
+        <origin xyz="0.33 0 0.075" rpy="0 0 0" />
         <axis   xyz="1 0 0" />
-        <limit  lower="0" upper="${pi/2}" velocity="100" effort="100"/>
+        <limit  lower="-${pi/18}" upper="${pi/18}" velocity="100" effort="100"/>
     </joint>
     <link name="Tool_link">

Commit message: update

File: urdf/robot_core.xacro (robot description, xacro)
@@ -1,12 +1,12 @@
 <?xml version="1.0"?>
 <robot xmlns:xacro="http://www.ros.org/wiki/xacro">
+     <link name="base_link">
+    </link>
+    <joint name="base_footprint_joint" type="fixed">
+        <parent link="base_link" />
+        <child  link="base_footprint" />
+        <origin xyz="0 0 -0.13" rpy="0 0 0"/>
+    </joint>
     <link name="base_footprint">
-    </link>
-    <joint name="base_link_joint" type="fixed">
-        <parent link="base_footprint" />
-        <child  link="base_link" />
-        <origin xyz="0 0 0.13" rpy="0 0 0"/>
-    </joint>
-    <link name="base_link">
     </link>
     <joint name="Chassis_joint" type="fixed">

Commit message: Update robot_core.xacro

File: urdf/robot_core.xacro (robot description, xacro)
@@ -88,5 +88,5 @@
     </link>
     <joint name="Tool_joint" type="revolute">
-        <parent link="base_link" />
+        <parent link="Chassis_link" />
         <child  link="Tool_link" />
         <origin xyz="0.33 0 0.075" rpy="0 0 0" />

Commit message: Update robot_core.xacro

File: urdf/robot_core.xacro (robot description, xacro)
@@ -88,7 +88,7 @@
     </link>
     <joint name="Tool_joint" type="revolute">
+        <origin xyz="0.33 0 0.075" rpy="0 0 0" />
         <parent link="Chassis_link" />
         <child  link="Tool_link" />
-        <origin xyz="0.33 0 0.075" rpy="0 0 0" />
         <axis   xyz="1 0 0" />
         <limit  lower="-${pi/18}" upper="${pi/18}" velocity="100" effort="100"/>

Commit message: Update robot_core.xacro

File: urdf/robot_core.xacro (robot description, xacro)
@@ -1,5 +1,5 @@
 <?xml version="1.0"?>
 <robot xmlns:xacro="http://www.ros.org/wiki/xacro">
-     <link name="base_link">
+    <link name="base_link">
     </link>
     <joint name="base_footprint_joint" type="fixed">
@@ -89,5 +89,5 @@
     <joint name="Tool_joint" type="revolute">
         <origin xyz="0.33 0 0.075" rpy="0 0 0" />
-        <parent link="Chassis_link" />
+        <parent link="base_link" />
         <child  link="Tool_link" />
         <axis   xyz="1 0 0" />

Commit message: Update robot_core.xacro

File: urdf/robot_core.xacro (robot description, xacro)
@@ -87,10 +87,10 @@
         </inertial>
     </link>
-    <joint name="Tool_joint" type="revolute">
+    <joint name="Tool_joint" type="fixed">
         <origin xyz="0.33 0 0.075" rpy="0 0 0" />
         <parent link="base_link" />
         <child  link="Tool_link" />
         <axis   xyz="1 0 0" />
-        <limit  lower="-${pi/18}" upper="${pi/18}" velocity="100" effort="100"/>
+        <!--<limit  lower="-${pi/18}" upper="${pi/18}" velocity="100" effort="100"/>  -->
     </joint>
     <link name="Tool_link">

Commit message: update

File: urdf/robot_core.xacro (robot description, xacro)
@@ -114,3 +114,53 @@
         </inertial>
     </link>
+    <joint name="LeftBrush_joint" type="fixed">
+        <origin xyz="0 -0.155 -0.073" rpy="0 0 0" />
+        <parent link="Tool_link" />
+        <child  link="LeftBrush_link" />
+    </joint>
+    <link name="LeftBrush_link">
+        <visual>
+            <origin xyz="0 0 0" rpy="0 0 0"/>
+            <geometry>
+                <mesh   filename="file://$(find AMR-Sweeper_description)/meshes/Tool/Brush.stl" />
+            </geometry>
+            <material name="red"/>
+        </visual>
+        <collision>
+            <origin xyz="0 0 0" rpy="0 0 0"/>
+            <geometry>
+                <mesh   filename="file://$(find AMR-Sweeper_description)/meshes/Tool/Brush.stl" />
+            </geometry>
+        </collision>
+        <inertial>
+            <origin xyz="0 0 0" rpy="0 0 0"/>
+            <mass value="1.5" />
+            <inertia ixx="0.01" ixy="0" ixz="0" iyy="0.02" iyz="0" izz="0.01" />
+        </inertial>
+    </link>
+    <joint name="RightBrush_joint" type="fixed">
+        <origin xyz="0 0.155 -0.073" rpy="0 0 0" />
+        <parent link="Tool_link" />
+        <child  link="RightBrush_link" />
+    </joint>
+    <link name="RightBrush_link">
+        <visual>
+            <origin xyz="0 0 0" rpy="0 0 0"/>
+            <geometry>
+                <mesh   filename="file://$(find AMR-Sweeper_description)/meshes/Tool/Brush.stl" />
+            </geometry>
+            <material name="red"/>
+        </visual>
+        <collision>
+            <origin xyz="0 0 0" rpy="0 0 0"/>
+            <geometry>
+                <mesh   filename="file://$(find AMR-Sweeper_description)/meshes/Tool/Brush.stl" />
+            </geometry>
+        </collision>
+        <inertial>
+            <origin xyz="0 0 0" rpy="0 0 0"/>
+            <mass value="1.5" />
+            <inertia ixx="0.01" ixy="0" ixz="0" iyy="0.02" iyz="0" izz="0.01" />
+        </inertial>
+    </link>
 </robot>

Commit message: update

File: urdf/robot_core.xacro (robot description, xacro)
@@ -54,5 +54,5 @@
             <origin xyz="0 0 0" rpy="${pi/2} 0 0"/>
             <geometry>
-                <cylinder radius="0.130" length="0.08"/>
+                <mesh   filename="file://$(find AMR-Sweeper_description)/meshes/WheelAssembly/WheelAssembly.stl" />
             </geometry>
         </collision>
@@ -80,5 +80,5 @@
             <origin xyz="0 0 0" rpy="${pi/2} 0 0"/>
             <geometry>
-                <cylinder radius="0.130" length="0.08"/>
+                <mesh   filename="file://$(find AMR-Sweeper_description)/meshes/WheelAssembly/WheelAssembly.stl" />
             </geometry>
         </collision>
