Commit message: Update IMU_sensor.xacro

File: urdf/IMU_sensor.xacro (robot description, xacro)
@@ -7,5 +7,5 @@
         <origin xyz="0.3 0 0.1" rpy="0 0 0"/>
     </joint>
-    <link name="GNSS_link">
+    <link name="IMU_link">
     </link>
 </robot>

Commit message: Update IMU_sensor.xacro

File: urdf/IMU_sensor.xacro (robot description, xacro)
@@ -8,4 +8,6 @@
     </joint>
     <link name="IMU_link">
+    </link>
+    <gazebo reference="IMU_link">
         <sensor name="imu_sensor" type="imu">
             <always_on>1</always_on>
@@ -14,4 +16,4 @@
             <topic>imu</topic>
         </sensor>
-    </link>
+    </gazebo>
 </robot>

Commit message: update

File: urdf/IMU_sensor.xacro (robot description, xacro)
@@ -8,4 +8,17 @@
     </joint>
     <link name="IMU_link">
+        <visual>
+            <origin xyz="0 0 0" rpy="0 0 0"/>
+            <geometry>
+                <box size="0.010 0.03 0.5"/>
+            </geometry>
+            <material name="black"/>
+        </visual>
+        <collision>
+            <origin xyz="0 0 0" rpy="0 0 0"/>
+            <geometry>
+                <box size="0.010 0.03 0.5"/>
+            </geometry>
+        </collision>
     </link>
     <gazebo reference="IMU_link">

File: urdf/depth_camera.xacro (robot description, xacro)
@@ -37,32 +37,5 @@
             </camera>
         </sensor>
-<!--         <sensor name="camera" type="depth_camera">
-            <camera>
-                <camera_info_topic>camera/camera_info</camera_info_topic>
-                <horizontal_fov>1.089</horizontal_fov>
-                <image>
-                    <width>640</width>
-                    <height>480</height>
-                    <format>B8G8R8</format>
-                </image>
-                <clip>
-                    <near>0.05</near>
-                    <far>8.0</far>
-                </clip>
-            </camera>
-            <always_on>1</always_on>
-            <update_rate>10</update_rate>
-            <visualize>true</visualize>
-            <topic>depth_camera</topic>
-       <plugin
-                filename="gz-sim-depth-camera-system"
-                name="gz::sim::systems::DepthCamera">
-                <gz_frame_id>camera_link_optical</gz_frame_id>
-                <min_depth>0.1</min_depth>
-                <max_depth>100.0</max_depth>
-            </plugin>
-     </sensor>
--->
-<!--        <sensor name="camera" type="camera">
+        <sensor name="camera" type="camera">
             <pose> 0 0 0 0 0 0 </pose>
             <visualize>true</visualize>
@@ -83,5 +56,4 @@
             <topic>camera/image_raw</topic>
         </sensor>
--->
     </gazebo>
 </robot>

Commit message: Update IMU_sensor.xacro

File: urdf/IMU_sensor.xacro (robot description, xacro)
@@ -3,22 +3,9 @@
 <!-- IMU Sensor -->
     <joint name="IMU_joint" type="fixed">
-        <parent link="base_link" />
+        <parent link="Tool_link" />
         <child  link="IMU_link" />
-        <origin xyz="0.3 0 0.1" rpy="0 0 0"/>
+        <origin xyz="0 0 0" rpy="0 0 0"/>
     </joint>
     <link name="IMU_link">
-        <visual>
-            <origin xyz="0 0 0" rpy="0 0 0"/>
-            <geometry>
-                <box size="0.010 0.03 0.5"/>
-            </geometry>
-            <material name="black"/>
-        </visual>
-        <collision>
-            <origin xyz="0 0 0" rpy="0 0 0"/>
-            <geometry>
-                <box size="0.010 0.03 0.5"/>
-            </geometry>
-        </collision>
     </link>
     <gazebo reference="IMU_link">

Commit message: Connect Tool_link to base_link

File: urdf/IMU_sensor.xacro (robot description, xacro)
@@ -1,12 +1,19 @@
 <?xml version="1.0"?>
 <robot xmlns:xacro="http://www.ros.org/wiki/xacro">
-<!-- IMU Sensor -->
-    <joint name="IMU_joint" type="fixed">
-        <parent link="Tool_link" />
-        <child  link="IMU_link" />
-        <origin xyz="0 0 0" rpy="0 0 0"/>
-    </joint>
-    <link name="IMU_link">
-    </link>
+<!-- Define Tool Link -->
+  <link name="Tool_link"/>
+  <!-- Connect Tool_link to base_link -->
+  <joint name="Tool_joint" type="fixed">
+      <parent link="base_link"/>
+      <child link="Tool_link"/>
+      <origin xyz="0.1 0 0.2" rpy="0 0 0"/>
+  </joint>
+  <!-- IMU Sensor -->
+  <joint name="IMU_joint" type="fixed">
+      <parent link="Tool_link" />
+      <child  link="IMU_link" />
+      <origin xyz="0 0 0" rpy="0 0 0"/>
+  </joint>
+  <link name="IMU_link"/>
     <gazebo reference="IMU_link">
         <sensor name="imu_sensor" type="imu">

Commit message: Update IMU_sensor.xacro

File: urdf/IMU_sensor.xacro (robot description, xacro)
@@ -1,13 +1,4 @@
 <?xml version="1.0"?>
 <robot xmlns:xacro="http://www.ros.org/wiki/xacro">
-<!-- Define Tool Link -->
-  <link name="Tool_link"/>
-  <!-- Connect Tool_link to base_link -->
-  <joint name="Tool_joint" type="fixed">
-      <parent link="base_link"/>
-      <child link="Tool_link"/>
-      <origin xyz="0.1 0 0.2" rpy="0 0 0"/>
-  </joint>
-  <!-- IMU Sensor -->
   <joint name="IMU_joint" type="fixed">
       <parent link="Tool_link" />

Commit message: Update IMU_sensor.xacro

File: urdf/IMU_sensor.xacro (robot description, xacro)
@@ -1,10 +1,12 @@
 <?xml version="1.0"?>
 <robot xmlns:xacro="http://www.ros.org/wiki/xacro">
-  <joint name="IMU_joint" type="fixed">
-      <parent link="Tool_link" />
-      <child  link="IMU_link" />
-      <origin xyz="0 0 0" rpy="0 0 0"/>
-  </joint>
-  <link name="IMU_link"/>
+<!-- IMU Sensor -->
+    <joint name="IMU_joint" type="fixed">
+        <parent link="Tool_link" />
+        <child  link="IMU_link" />
+        <origin xyz="0 0 0" rpy="0 0 0"/>
+    </joint>
+    <link name="IMU_link">Add commentMore actions
+    </link>
     <gazebo reference="IMU_link">
         <sensor name="imu_sensor" type="imu">
