Commit message: GNSS .stl included in code

File: urdf/GNSS_sensor.xacro (robot description, xacro)
@@ -5,5 +5,5 @@
         <parent link="base_link" />
         <child  link="GNSS_link" />
-        <origin xyz="0 0 0.2" rpy="0 0 0"/>
+        <origin xyz="0 0 0.199" rpy="0 0 0"/>
     </joint>
     <link name="GNSS_link">
@@ -11,6 +11,5 @@
             <origin xyz="0 0 0" rpy="0 0 0"/>
             <geometry>
-            <!--    <mesh   filename="file://$(find AMR-Sweeper_description)/meshes/Sensors/GNSS.stl" />  -->
-            <box size="0.010 0.03 0.03"/>
+            <mesh   filename="file://$(find AMR-Sweeper_description)/meshes/Sensors/GNSS.stl" />
             </geometry>
             <material name="black"/>
@@ -19,6 +18,5 @@
             <origin xyz="0 0 0" rpy="0 0 0"/>
             <geometry>
-            <!--    <mesh   filename="file://$(find AMR-Sweeper_description)/meshes/Sensors/GNSS.stl" />  -->
-            <box size="0.010 0.03 0.03"/>
+            <mesh   filename="file://$(find AMR-Sweeper_description)/meshes/Sensors/GNSS.stl" />
             </geometry>
         </collision>

Commit message: Update GNSS_sensor.xacro
update

File: urdf/GNSS_sensor.xacro (robot description, xacro)
@@ -24,5 +24,5 @@
             <origin xyz="0 0 0" rpy="0 0 0"/>
             <mass value="0" />
-            <inertia ixx="0" ixy="0" ixz="0" iyy="0" iyz="0" izz="0" />
+        <!--    <inertia ixx="0" ixy="0" ixz="0" iyy="0" iyz="0" izz="0" /> -->
         </inertial>
     </link>

Commit message: update

File: urdf/GNSS_sensor.xacro (robot description, xacro)
@@ -21,9 +21,4 @@
             </geometry>
         </collision>
-        <inertial>
-            <origin xyz="0 0 0" rpy="0 0 0"/>
-            <mass value="0" />
-        <!--    <inertia ixx="0" ixy="0" ixz="0" iyy="0" iyz="0" izz="0" /> -->
-        </inertial>
     </link>
 <gazebo reference="GNSS_link">

Commit message: update

File: urdf/GNSS_sensor.xacro (robot description, xacro)
@@ -15,10 +15,4 @@
             <material name="black"/>
         </visual>
-        <collision>
-            <origin xyz="0 0 0" rpy="0 0 0"/>
-            <geometry>
-            <mesh   filename="file://$(find AMR-Sweeper_description)/meshes/Sensors/GNSS.stl" />
-            </geometry>
-        </collision>
     </link>
 <gazebo reference="GNSS_link">

Commit message: Update GNSS_sensor.xacro

File: urdf/GNSS_sensor.xacro (robot description, xacro)
@@ -11,5 +11,5 @@
             <origin xyz="0 0 0" rpy="0 0 0"/>
             <geometry>
-            <mesh   filename="file://$(find AMR-Sweeper_description)/meshes/Sensors/GNSS.stl" />
+            <mesh   filename="package://AMR-Sweeper_description/meshes/Sensors/GNSS.stl" />
             </geometry>
             <material name="black"/>

Commit message: Use find with pkg name

File: urdf/GNSS_sensor.xacro (robot description, xacro)
@@ -11,5 +11,5 @@
             <origin xyz="0 0 0" rpy="0 0 0"/>
             <geometry>
-            <mesh   filename="package://AMR-Sweeper_description/meshes/Sensors/GNSS.stl" />
+            <mesh   filename="$(find amr_sweeper_description)/meshes/Sensors/GNSS.stl" />
             </geometry>
             <material name="black"/>

File: urdf/robot_core.xacro (robot description, xacro)
@@ -19,5 +19,5 @@
             <origin xyz="0 0 0" rpy="0 0 0"/>
             <geometry>
-                <mesh   filename="package://AMR-Sweeper_description/meshes/Chassis/Chassis.stl" />
+                <mesh   filename="$(find amr_sweeper_description)/meshes/Chassis/Chassis.stl" />
             </geometry>
             <material name="grey"/>
@@ -27,5 +27,5 @@
             <origin xyz="0 0 0" rpy="0 0 0"/>
             <geometry>
-                <mesh   filename="package://AMR-Sweeper_description/meshes/Chassis/Chassis.stl" />
+                <mesh   filename="$(find amr_sweeper_description)/meshes/Chassis/Chassis.stl" />
             </geometry>
         </collision>
@@ -47,5 +47,5 @@
             <origin xyz="0 0 0" rpy="${pi/2} 0 0"/>
             <geometry>
-                <mesh   filename="package://AMR-Sweeper_description/meshes/WheelAssembly/WheelAssembly.stl" />
+                <mesh   filename="$(find amr_sweeper_description)/meshes/WheelAssembly/WheelAssembly.stl" />
             </geometry>
             <material name="yellow"/>
@@ -54,5 +54,5 @@
             <origin xyz="0 0 0" rpy="${pi/2} 0 0"/>
             <geometry>
-                <mesh   filename="package://AMR-Sweeper_description/meshes/WheelAssembly/WheelAssembly.stl" />
+                <mesh   filename="$(find amr_sweeper_description)/meshes/WheelAssembly/WheelAssembly.stl" />
             </geometry>
         </collision>
@@ -73,5 +73,5 @@
             <origin xyz="0 0 0" rpy="${pi/2} 0 0"/>
             <geometry>
-                <mesh   filename="package://AMR-Sweeper_description/meshes/WheelAssembly/WheelAssembly.stl" />
+                <mesh   filename="$(find amr_sweeper_description)/meshes/WheelAssembly/WheelAssembly.stl" />
             </geometry>
             <material name="yellow"/>
@@ -80,5 +80,5 @@
             <origin xyz="0 0 0" rpy="${pi/2} 0 0"/>
             <geometry>
-                <mesh   filename="package://AMR-Sweeper_description/meshes/WheelAssembly/WheelAssembly.stl" />
+                <mesh   filename="$(find amr_sweeper_description)/meshes/WheelAssembly/WheelAssembly.stl" />
             </geometry>
         </collision>
@@ -100,5 +100,5 @@
             <origin xyz="0 0 0" rpy="0 0 0"/>
             <geometry>
-                <mesh   filename="package://AMR-Sweeper_description/meshes/Tool/Tool.stl" />
+                <mesh   filename="$(find amr_sweeper_description)/meshes/Tool/Tool.stl" />
             </geometry>
             <material name="black"/>
@@ -119,5 +119,5 @@
             <origin xyz="0 0 0" rpy="0 0 0"/>
             <geometry>
-                <mesh   filename="package://AMR-Sweeper_description/meshes/Tool/Brush.stl" />
+                <mesh   filename="$(find amr_sweeper_description)/meshes/Tool/Brush.stl" />
             </geometry>
             <material name="red"/>
@@ -126,5 +126,5 @@
             <origin xyz="0 0 0" rpy="0 0 0"/>
             <geometry>
-                <mesh   filename="package://AMR-Sweeper_description/meshes/Tool/Brush.stl" />
+                <mesh   filename="$(find amr_sweeper_description)/meshes/Tool/Brush.stl" />
             </geometry>
         </collision>
@@ -144,5 +144,5 @@
             <origin xyz="0 0 0" rpy="0 0 0"/>
             <geometry>
-                <mesh   filename="package://AMR-Sweeper_description/meshes/Tool/Brush.stl" />
+                <mesh   filename="$(find amr_sweeper_description)/meshes/Tool/Brush.stl" />
             </geometry>
             <material name="red"/>
@@ -151,5 +151,5 @@
             <origin xyz="0 0 0" rpy="0 0 0"/>
             <geometry>
-                <mesh   filename="package://AMR-Sweeper_description/meshes/Tool/Brush.stl" />
+                <mesh   filename="$(find amr_sweeper_description)/meshes/Tool/Brush.stl" />
             </geometry>
         </collision>
